File: HardWare/CW32_Lightmeter.kicad_sch (KiCad schematic)
At the start: 42 parts, among them J1 USB_C_Receptacle, SW1 TM-2022-3, SW2 Power_KEY, U1 CW32F030C8T6, U3 BH1750FVI-TR, U4 TP4055, U5 EC190707, U6 RT9013-33GB, U7 CH340G, X1 X1E0000210375000G

Commit message: Update PCB Layout
Parts:
- removed U7: CH340G, Package_SO:SOIC-16_3.9x9.9mm_P1.27mm, symbol Interface_USB:CH340G
- added C1, C2: 0.1uF, Capacitor_SMD:C_0603_1608Metric, symbol Device:C
- added C3, C4: 2.2pF, Capacitor_SMD:C_0603_1608Metric, symbol Device:C
- added J2: Conn_01x04_Pin, Userlib:SWD_Port, symbol Connector:Conn_01x04_Pin
- added R15: 1MR, Resistor_SMD:R_0603_1608Metric, symbol Device:R
- added U2: CH340C, Package_SO:SOIC-16_3.9x9.9mm_P1.27mm, symbol Interface_USB:CH340C
- X1: value X1E0000210375000G -> 12MHz
Connections:
- net +3.3VA is gone; now on net +3.3V: U1.9 (VDDA)
- net +3.3V: now also C2.2, J2.1 (Pin_1), U2.16 (VCC)
- net GND: now also C1.1, C2.1, C3.2, C4.1, J2.4 (Pin_4), U2.1 (GND)
- net SWCLK: now also J2.2 (Pin_2)
- net SWDIO: now also J2.3 (Pin_3)
- net USB_DN: now also U2.6 (UD-)
- net USB_DP: now also U2.5 (UD+)
- net at U1.5 (PF0-OSC_IN), X1.1 (OSC1): now also C4.2, R15.1
- net at U1.6 (PF1-OSC_OUT), X1.3 (OSC2): now also C3.1, R15.2
- net UART3_TX: now reaches U1.12 (PA2)
- net UART3_TX: now also U2.3 (RXD)
- net UART3_RX: now reaches U1.13 (PA3)
- net UART3_RX: now also U2.2 (TXD)
- new net: C1.2, U2.4 (V3)
- no-connect marks 15 -> 20
Other:
- moved on the sheet: C12, C13, C14, R1, SW1, U1

Commit message: Update PCB Layout
Parts:
- added C20: 10uF, Capacitor_SMD:C_0603_1608Metric, symbol Device:C
- added R16: 1KR, Resistor_SMD:R_0603_1608Metric, symbol Device:R
Connections:
- net +3.3V: now also R16.2
- net GND: now also C20.2
- net NRST: now also C20.1, R16.1
- net SW_Down: now also SW1.d, U1.18 (PB0); no longer SW1.b, U1.19 (PB1)
- net SW_UP: now also SW1.b; no longer SW1.d
- net SW_Power renamed SW_Enter
- net SW_Enter: now also U1.19 (PB1)
Other:
- moved on the sheet: J2

Commit message: Update PCB Layout
Connections:
- net SWCLK: now also J2.3 (Pin_3); no longer J2.2 (Pin_2)
- net SWDIO: now also J2.2 (Pin_2); no longer J2.3 (Pin_3)
Changed lines of the file:
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@@
     (fill (type none))
+  )
+  (label "SWCLK" (at 159.766 58.928 180) (fields_autoplaced)
+    (effects (font (size 1.27 1.27)) (justify right bottom))
   )
   (label "SW_UP" (at 42.672 82.296 0) (fields_autoplaced)
     (effects (font (size 1.27 1.27)) (justify left bottom))
+  )
+  (label "SWDIO" (at 159.766 56.388 180) (fields_autoplaced)
+    (effects (font (size 1.27 1.27)) (justify right bottom))
   )
   (label "UART3_RX" (at 387.35 65.786 180) (fields_autoplaced)
@@
   (label "NRST" (at 48.26 49.276 0) (fields_autoplaced)
     (effects (font (size 1.27 1.27)) (justify left bottom))
-  )
-  (label "SWCLK" (at 159.766 56.388 180) (fields_autoplaced)
-    (effects (font (size 1.27 1.27)) (justify right bottom))
   )
   (label "USB_DN" (at 337.566 38.862 180) (fields_autoplaced)
@@
     (effects (font (size 1.27 1.27)) (justify left bottom))
   )
-  (label "SWDIO" (at 159.766 58.928 180) (fields_autoplaced)
-    (effects (font (size 1.27 1.27)) (justify right bottom))
-  )
   (label "BH1750_SCL" (at 261.62 137.414 180) (fields_autoplaced)

Commit message: Finished PCB Layout
Parts:
- added R17, R18, R19, R20: 4K7, Resistor_SMD:R_0603_1608Metric, symbol Device:R
Connections:
- net +3.3V: now also R17.1, R18.1, R19.1, R20.1
- net BH1750_SCL: now also R17.2
- net BH1750_SDA: now also R18.2
- net OLED_SCL: now also U1.26 (PB13), R19.2
- net OLED_SDA: now also U1.27 (PB14), R20.2
