File: HardWare/CW32_Lightmeter.kicad_pcb (KiCad board)
At the start: 2 copper layers, 47 parts, among them J1 USB_C_Receptacle, SW1 TM-2022-3, SW2 Power_KEY, U1 CW32F030C8T6, U2 AMS1117-3.3, U3 BH1750FVI-TR, U4 TP4055, U5 EC190707, U6 RT9013-33GB, U7 CH340G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

Commit message: Update SCH
Parts:
- removed C1, C4: 0.1uF, Capacitor_SMD:C_0603_1608Metric
- removed C2, C3: 10uF, Capacitor_SMD:C_0603_1608Metric
- removed U2: AMS1117-3.3, Package_TO_SOT_SMD:SOT-223-3_TabPin2
- moved X1 41.1 mm to (49.1, 64.7)
- moved SW2 36.0 mm to (52.1, 47.7)
- moved U6 34.7 mm to (37.0, 63.2)
- moved U4 34.0 mm to (41.4, 63.2)
- moved U1 32.3 mm to (60.2, 56.5)
- moved U5 32.2 mm to (62.9, 64.2)
- moved U3 32.1 mm to (57.3, 66.8)
- moved SW1 27.4 mm to (27.4, 61.7)
- moved C6 17.6 mm to (50.6, 21.4)
- moved C7 17.6 mm to (50.6, 23.9)
- moved C8 17.6 mm to (50.6, 26.5)
- moved C5 17.6 mm to (50.6, 18.9)
- moved C9 17.6 mm to (50.6, 29.0)
- moved J1 17.5 mm to (40.4, 56.3)
- moved U7 15.8 mm to (50.4, 56.7)
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
Commit message: Update PCB Layout
Parts:
- removed U7: CH340G, Package_SO:SOIC-16_3.9x9.9mm_P1.27mm
- added C1: 0.1uF, Capacitor_SMD:C_0603_1608Metric, F.Cu at (51.5, 103.2)
- added C2: 0.1uF, Capacitor_SMD:C_0603_1608Metric, F.Cu at (60.6, 100.7)
- added C3: 2.2pF, Capacitor_SMD:C_0603_1608Metric, F.Cu at (45.3, 106.3)
- added C4: 2.2pF, Capacitor_SMD:C_0603_1608Metric, F.Cu at (39.2, 106.4)
- added J2: Conn_01x04_Pin, Userlib:SWD_Port, F.Cu at (62.9, 89.7)
- added R15: 1MR, Resistor_SMD:R_0603_1608Metric, F.Cu at (42.4, 109.2)
- added U2: CH340C, Package_SO:SOIC-16_3.9x9.9mm_P1.27mm, F.Cu at (56.1, 104.4)
- D2, U3: moved to B.Cu
- X1: value X1E0000210375000G -> 12MHz
- moved R10 102.1 mm to (38.6, 118.2)
- moved C15 94.9 mm to (29.9, 115.5), turned to 90 degrees
- moved R11 90.0 mm to (44.7, 109.6), turned to 90 degrees
- moved C16 88.4 mm to (32.4, 112.0), turned to 180 degrees
- moved R7 87.3 mm to (34.8, 115.5), turned to 90 degrees
- moved R12 86.1 mm to (50.4, 109.1), turned to -90 degrees
- moved C18 85.9 mm to (36.4, 115.4), turned to -90 degrees
- moved R9 85.3 mm to (32.4, 117.7), turned to 180 degrees
- moved C14 85.0 mm to (46.9, 106.1), turned to -90 degrees
- moved C17 84.2 mm to (57.1, 113.1)
- moved R13 83.8 mm to (48.9, 109.1), turned to 90 degrees
- moved R8 83.6 mm to (29.9, 112.5), turned to 90 degrees
- moved R14 81.6 mm to (47.3, 109.1), turned to 90 degrees
- moved C19 80.2 mm to (38.5, 112.6), turned to 180 degrees
- moved C13 76.6 mm to (51.4, 95.5), turned to -90 degrees
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Connections:
- U1 pad 12: unconnected-(U1-PA2-Pad12) -> /UART3_TX
- U1 pad 13: unconnected-(U1-PA3-Pad13) -> /UART3_RX
- U1 pad 9: +3.3VA -> +3.3V
Other:
- board outline added: 35 x 37.3 mm

Commit message: Update PCB Layout
Parts:
- added C20: 10uF, Capacitor_SMD:C_0603_1608Metric, F.Cu at (47.6, 105.9)
- added R16: 1KR, Resistor_SMD:R_0603_1608Metric, F.Cu at (49.1, 105.9)
- moved C14 3.74 mm to (50.6, 105.9)
- moved C1 2.79 mm to (52.2, 105.9), turned to 90 degrees
- moved D2 2.52 mm to (32.4, 112.0)
- moved C2 1.83 mm to (61.2, 102.4)
- moved U2 1.83 mm to (56.7, 106.1)
- moved R13 1.45 mm to (47.5, 109.6)
- moved R12 1.45 mm to (49.0, 109.6), turned to 90 degrees
- moved R14 1.45 mm to (46.0, 109.6)
- moved C13 1.05 mm to (50.7, 94.7), turned to 0 degrees
- moved C17 1.03 mm to (56.1, 112.7)
- moved U3 1.02 mm to (31.1, 85.6)
- moved C15 1.00 mm to (29.9, 116.5)
- moved R8 1.00 mm to (29.9, 113.5)
- moved C5 0.97 mm to (32.2, 85.7)
- moved C6 0.97 mm to (30.6, 85.7)
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Connections:
- SW1 pad b: /SW_Down -> /SW_UP
- SW1 pad c: /SW_Power -> /SW_Enter
- SW1 pad d: /SW_UP -> /SW_Down
- U1 pad 18: unconnected-(U1-PB0-Pad18) -> /SW_Down
- U1 pad 19: /SW_Down -> /SW_Enter
Routing:
- net +3.3V: track 0.00 -> 25.8 mm
- net /SW_Down: track 0.00 -> 14.6 mm, vias 0 -> 2
- net /SW_UP: track 0.00 -> 14.1 mm, vias 0 -> 2
- net /SW_Enter: track 0.00 -> 13.5 mm, vias 0 -> 2
- net Net-(D1-A): track 0.00 -> 11.2 mm
- net Net-(U1-PF0-OSC_IN): track 0.00 -> 11.1 mm
- net /USB_DP: track 0.00 -> 9.23 mm
- net Net-(U1-PF1-OSC_OUT): track 0.00 -> 8.41 mm
- net /USB_DN: track 0.00 -> 7.89 mm
- net GND: track 0.00 -> 7.25 mm
- net /UART3_TX: track 0.00 -> 7.25 mm
- net Net-(OLED1-D/C#): track 0.00 -> 6.19 mm
- net Net-(J1-D+-PadA6): track 0.00 -> 5.58 mm, vias 0 -> 2
- net /UART3_RX: track 0.00 -> 5.48 mm
- net Net-(OLED1-C1N): track 0.00 -> 4.50 mm
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
Commit message: Update PCB Layout
Connections:
- J2 pad 2: /SWCLK -> /SWDIO
- J2 pad 3: /SWDIO -> /SWCLK
Routing:
- net +5V: track 0.00 -> 34.3 mm, vias 0 -> 2
- net /BAT_EN: track 0.00 -> 19.2 mm
- net +BATT: track 0.00 -> 10.1 mm
- net Net-(U4-VCC): track 0.00 -> 5.91 mm
- net +3.3V: track 25.8 -> 29.5 mm
- net GND: track 7.25 -> 9.97 mm
- net Net-(U4-PROG): track 0.00 -> 1.62 mm
Changed lines of the file:
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@@
       (net 6 "+3.3V") (pinfunction "Pin_1") (pintype "passive") (thermal_bridge_angle 45))
     (pad "2" smd roundrect (at -0.52 -0.5 90) (size 1 1) (layers "F.Cu" "F.Paste" "F.Mask") (roundrect_rratio 0.1)
-      (net 57 "/SWCLK") (pinfunction "Pin_2") (pintype "passive") (thermal_bridge_angle 45))
+      (net 56 "/SWDIO") (pinfunction "Pin_2") (pintype "passive") (thermal_bridge_angle 45))
     (pad "3" smd roundrect (at 0.6 -0.5 90) (size 1 1) (layers "F.Cu" "F.Paste" "F.Mask") (roundrect_rratio 0.1)
-      (net 56 "/SWDIO") (pinfunction "Pin_3") (pintype "passive") (thermal_bridge_angle 45))
+      (net 57 "/SWCLK") (pinfunction "Pin_3") (pintype "passive") (thermal_bridge_angle 45))
     (pad "4" smd roundrect (at 1.72 -0.5 90) (size 1 1) (layers "F.Cu" "F.Paste" "F.Mask") (roundrect_rratio 0.1)
       (net 5 "GND") (pinfunction "Pin_4") (pintype "passive") (thermal_bridge_angle 45))
@@
   (gr_rect (start 28.32 82.4) (end 63.3 119.72)
     (stroke (width 0.1) (type default)) (fill none) (layer "Edge.Cuts"))
+  (segment (start 33.265 117.67) (end 33.235 117.64) (width 0.3) (layer "F.Cu") (net 1))
+  (segment (start 55.341 112.73) (end 52.89 112.73) (width 0.3) (layer "F.Cu") (net 1))
+  (segment (start 48.96 111.19) (end 48.43 111.72) (width 0.3) (layer "F.Cu") (net 1))
+  (segment (start 43.63 113.011827) (end 44.528173 113.91) (width 0.3) (layer "F.Cu") (net 1))
+  (segment (start 34.42 117.67) (end 33.265 117.67) (width 0.3) (layer "F.Cu") (net 1))
+  (segment (start 43.63 112.26) (end 43.63 111.76) (width 0.3) (layer "F.Cu") (net 1))
+  (segment (start 47.531827 113.91) (end 48.43 113.011827) (width 0.3) (layer "F.Cu") (net 1))
+  (segment (start 56.23 113.619) (end 55.341 112.73) (width 0.3) (layer "F.Cu") (net 1))
+  (segment (start 35.49 111.16) (end 34.91 111.74) (width 0.3) (layer "F.Cu") (net 1))
+  (segment (start 34.91 111.74) (end 34.91 111.75) (width 0.3) (layer "F.Cu") (net 1))
+  (segment (start 56.23 114.22) (end 56.23 113.619) (width 0.3) (layer "F.Cu") (net 1))
+  (segment (start 43.63 112.26) (end 43.63 113.011827) (width 0.3) (layer "F.Cu") (net 1))
+  (segment (start 48.43 113.011827) (end 48.43 112.26) (width 0.3) (layer "F.Cu") (net 1))
+  (segment (start 43.03 111.16) (end 35.49 111.16) (width 0.3) (layer "F.Cu") (net 1))
+  (segment (start 34.91 111.75) (end 34.89 111.77) (width 0.3) (layer "F.Cu") (net 1))
+  (segment (start 48.43 111.72) (end 48.43 112.26) (width 0.3) (layer "F.Cu") (net 1))
+  (segment (start 52.89 112.73) (end 51.35 111.19) (width 0.3) (layer "F.Cu") (net 1))
+  (segment (start 51.35 111.19) (end 48.96 111.19) (width 0.3) (layer "F.Cu") (net 1))
+  (segment (start 43.63 111.76) (end 43.03 111.16) (width 0.3) (layer "F.Cu") (net 1))
+  (segment (start 44.528173 113.91) (end 47.531827 113.91) (width 0.3) (layer "F.Cu") (net 1))
+  (via (at 34.42 117.67) (size 0.45) (drill 0.3) (layers "F.Cu" "B.Cu") (net 1))
+  (via (at 34.89 111.77) (size 0.45) (drill 0.3) (layers "F.Cu" "B.Cu") (net 1))
+  (segment (start 34.89 111.77) (end 34.89 117.2) (width 0.3) (layer "B.Cu") (net 1))
+  (segment (start 34.89 117.2) (end 34.42 117.67) (width 0.3) (layer "B.Cu") (net 1))
   (segment (start 44.124 107.025) (end 45.735 107.025) (width 0.15) (layer "F.Cu") (net 5))
   (segment (start 52.16 106.695) (end 50.62 106.695) (width 0.15) (layer "F.Cu") (net 5))
+  (segment (start 49.775 112.26) (end 50.35 112.835) (width 0.3) (layer "F.Cu") (net 5))
   (segment (start 41.924 105.325) (end 40.055 105.325) (width 0.15) (layer "F.Cu") (net 5))
+  (segment (start 49.23 112.26) (end 49.775 112.26) (width 0.3) (layer "F.Cu") (net 5))
   (segment (start 47.575 106.7) (end 47.58 106.695) (width 0.15) (layer "F.Cu") (net 5))
   (segment (start 46.06 106.7) (end 47.575 106.7) (width 0.15) (layer "F.Cu") (net 5))
   (segment (start 45.735 107.025) (end 46.06 106.7) (width 0.15) (layer "F.Cu") (net 5))
+  (segment (start 42.83 112.26) (end 42.285 112.26) (width 0.3) (layer "F.Cu") (net 5))
+  (segment (start 42.285 112.26) (end 41.71 112.835) (width 0.3) (layer "F.Cu") (net 5))
   (segment (start 40.055 105.325) (end 39.88 105.15) (width 0.15) (layer "F.Cu") (net 5))
   (segment (start 49.1 105.095) (end 50.57 105.095) (width 0.15) (layer "F.Cu") (net 6))
@@
   (segment (start 48.255 96.155) (end 49.29 96.155) (width 0.15) (layer "F.Cu") (net 6))
   (segment (start 49.905 94.69) (end 49.29 95.305) (width 0.15) (layer "F.Cu") (net 6))
+  (segment (start 37.9105 114.26475) (end 37.91 114.26525) (width 0.3) (layer "F.Cu") (net 6))
   (segment (start 42.6 102.23) (end 46.04 102.23) (width 0.15) (layer "F.Cu") (net 6))
   (segment (start 50.57 105.095) (end 50.62 105.145) (width 0.15) (layer "F.Cu") (net 6))
   (segment (start 42.29 103.155) (end 42.29 102.54) (width 0.15) (layer "F.Cu") (net 6))
   (segment (start 46.821594 104.24) (end 46.29 103.708406) (width 0.15) (layer "F.Cu") (net 6))
+  (segment (start 37.9105 112.6) (end 37.9105 114.26475) (width 0.3) (layer "F.Cu") (net 6))
   (segment (start 40.79 102.82) (end 40.79 101.655) (width 0.15) (layer "F.Cu") (net 6))
   (segment (start 40.465 103.155) (end 42.29 103.155) (width 0.15) (layer "F.Cu") (net 6))
+  (segment (start 59.235 101.625) (end 59.18 101.68) (width 0.3) (layer "F.Cu") (net 6))
   (segment (start 46.29 103.708406) (end 46.29 103.155) (width 0.15) (layer "F.Cu") (net 6))
   (segment (start 47.44 100.83) (end 47.44 96.96) (width 0.15) (layer "F.Cu") (net 6))
+  (segment (start 61.24 101.625) (end 59.235 101.625) (width 0.3) (layer "F.Cu") (net 6))
   (segment (start 48.25 96.15) (end 48.255 96.155) (width 0.15) (layer "F.Cu") (net 6))
   (segment (start 50.62 105.145) (end 49.715 104.24) (width 0.15) (layer "F.Cu") (net 6))
@@
   (segment (start 47.58 105.225) (end 49.1 106.745) (width 0.15) (layer "F.Cu") (net 53))
   (segment (start 47.58 105.145) (end 47.58 105.225) (width 0.15) (layer "F.Cu") (net 53))
+  (segment (start 29.85 117.32) (end 31.265 117.32) (width 0.3) (layer "F.Cu") (net 59))
+  (segment (start 31.346 115.811) (end 29.85 114.315) (width 0.3) (layer "F.Cu") (net 59))
+  (segment (start 31.346 116.21) (end 31.346 115.811) (width 0.3) (layer "F.Cu") (net 59))
+  (segment (start 31.346 116.21) (end 31.346 117.401) (width 0.3) (layer "F.Cu") (net 59))
+  (segment (start 31.346 117.401) (end 31.585 117.64) (width 0.3) (layer "F.Cu") (net 59))
+  (segment (start 31.265 117.32) (end 31.585 117.64) (width 0.3) (layer "F.Cu") (net 59))
+  (segment (start 31.346 114.596) (end 31.91 115.16) (width 0.3) (layer "F.Cu") (net 60))
+  (segment (start 31.346 112.309) (end 31.635 112.02) (width 0.3) (layer "F.Cu") (net 60))
+  (segment (start 34.34 115.46) (end 35.655 115.46) (width 0.3) (layer "F.Cu") (net 60))
+  (segment (start 35.655 115.46) (end 36.41 116.215) (width 0.3) (layer "F.Cu") (net 60))
+  (segment (start 37.91 116.57325) (end 36.76825 116.57325) (width 0.3) (layer "F.Cu") (net 60))
+  (segment (start 36.76825 116.57325) (end 36.41 116.215) (width 0.3) (layer "F.Cu") (net 60))
+  (segment (start 31.91 115.16) (end 34.04 115.16) (width 0.3) (layer "F.Cu") (net 60))
+  (segment (start 31.346 113.61) (end 31.346 112.309) (width 0.3) (layer "F.Cu") (net 60))
+  (segment (start 31.346 113.61) (end 31.346 114.596) (width 0.3) (layer "F.Cu") (net 60))
+  (segment (start 34.04 115.16) (end 34.34 115.46) (width 0.3) (layer "F.Cu") (net 60))
+  (segment (start 33.311 116.275) (end 33.246 116.21) (width 0.3) (layer "F.Cu") (net 62))
+  (segment (start 34.835 116.275) (end 33.311 116.275) (width 0.3) (layer "F.Cu") (net 62))
+  (segment (start 54.43 118.52) (end 41.44 118.52) (width 0.15) (layer "F.Cu") (net 64))
+  (segment (start 41.44 118.52) (end 39.81 116.89) (width 0.15) (layer "F.Cu") (net 64))
+  (segment (start 39.81 116.89) (end 39.81 116.57325) (width 0.15) (layer "F.Cu") (net 64))
+  (segment (start 55.28 117.67) (end 54.43 118.52) (width 0.15) (layer "F.Cu") (net 64))
+  (segment (start 39.5105 118.17) (end 39.5105 116.87275) (width 0.3) (layer "F.Cu") (net 64))
+  (segment (start 55.28 117.02) (end 55.28 117.67) (width 0.15) (layer "F.Cu") (net 64))
+  (segment (start 39.5105 116.87275) (end 39.81 116.57325) (width 0.3) (layer "F.Cu") (net 64))
   (segment (start 44.78 111.1) (end 44.78 112.26) (width 0.15) (layer "F.Cu") (net 69))
   (segment (start 44.44 110.76) (end 44.78 111.1) (width 0.15) (layer "F.Cu") (net 69))

Commit message: Finished PCB Layout
Parts:
- added R17: 4K7, Resistor_SMD:R_0603_1608Metric, F.Cu at (53.1, 98.9)
- added R18: 4K7, Resistor_SMD:R_0603_1608Metric, F.Cu at (53.1, 97.4)
- added R19: 4K7, Resistor_SMD:R_0603_1608Metric, F.Cu at (48.3, 93.1)
- added R20: 4K7, Resistor_SMD:R_0603_1608Metric, F.Cu at (45.2, 93.1)
Connections:
- U1 pad 26: unconnected-(U1-PB13-Pad26) -> /OLED_SCL
- U1 pad 27: unconnected-(U1-PB14-Pad27) -> /OLED_SDA
Routing:
- net +3.3V: track 29.5 -> 121.4 mm, vias 0 -> 7
- net GND: track 9.97 -> 62.2 mm, vias 0 -> 12
- net /BH1750_SCL: track 0.00 -> 50.0 mm, vias 0 -> 3
- net /BH1750_SDA: track 0.00 -> 48.0 mm, vias 0 -> 3
- net Net-(U5-KEY): track 0.00 -> 29.9 mm
- net /SWCLK: track 0.00 -> 24.6 mm, vias 0 -> 2
- net /SWDIO: track 0.00 -> 23.6 mm, vias 0 -> 2
- net /OLED_SCL: track 0.00 -> 8.89 mm, vias 0 -> 2
- net /OLED_SDA: track 0.00 -> 8.47 mm, vias 0 -> 2
- net /NRST: track 2.23 -> 5.68 mm
- net Net-(D2-K): track 0.00 -> 2.62 mm, vias 0 -> 1
- net Net-(D2-A): track 0.00 -> 2.24 mm, vias 0 -> 1
- net Net-(U3-DVI): track 0.00 -> 2.00 mm, vias 0 -> 1
- added copper zone on B.Cu, net GND
- added copper zone on F.Cu, net GND
Other:
- board text added: "0"
- board text added: "0 mm"
- board text added: "0.01 mm"
- board text added: "0.02"
- board text added: "0.035 mm"
- board text added: "1"
- board text added: "1.51 mm"
- board text added: "3.3"
- board text added: "4.5"
- board text added: "B.Cu"
- board text added: "B.Mask"
- board text added: "B.Paste"
- board text added: "B.Silkscreen"
- board text added: "Bottom Silk Screen"
- board text added: "Bottom Solder Mask"
- board text added: "Bottom Solder Paste"
- board text added: "Epsilon R（相对介电常数）"
- board text added: "F.Cu"
- board text added: "F.Mask"
- board text added: "F.Paste"
- board text added: "F.Silkscreen"
- board text added: "FR4"
- board text added: "Loss Tangent（损耗角正切）"
- board text added: "Not specified"
- board text added: "Top Silk Screen"
- board text added: "Top Solder Mask"
- board text added: "Top Solder Paste"
- board text added: "copper"
- board text added: "core"
- board text added: "层名称"
- board text added: "材料"
- board text added: "电介质"
- board text added: "类型"
- board text added: "线宽 (mm)"
- board text added: "颜色"

Commit message: Hardware Finished
Parts:
- added REF**: MountingHole_2.2mm_M2_DIN965_Pad_TopBottom, MountingHole:MountingHole_2.2mm_M2_DIN965_Pad_TopBottom, F.Cu at (32.5, 108.6)
- added REF**: MountingHole_2.2mm_M2_DIN965_Pad_TopBottom, MountingHole:MountingHole_2.2mm_M2_DIN965_Pad_TopBottom, F.Cu at (60.0, 113.6)
Other:
- outline, holes or cut-outs redrawn
